File: unchat_keeb/unchat_keeb.kicad_pcb (KiCad board)
At the start: 2 copper layers, 274 x 102 mm, 299 parts, among them U1 74HC365, U10 74HC14, U11 74HC14, U12 74HC14, U13 74HC174, U14 74HC174, U15 74HC174, U16 74HC174, U17 74HC174, U18 74HC174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

Commit message: Remove pullups, as RPi GPIOs are pulled by default
Parts:
- removed R129, R130, R131, R132, R133, R134: 1k, Resistor_SMD:R_0805_2012Metric
