File: unchat_keeb/led_control.kicad_sch (KiCad schematic)
At the start: 2 parts, among them U14 74HC174, U19 74HC365

Commit message: Add dxf layout and finish half keyboard pbc layout
Connections:
- net BUS1: now also U14.6 (D2); no longer U14.3 (D0)
- net BUS3: now also U14.3 (D0); no longer U14.6 (D2)
- net BUS4: now also U14.14 (D5); no longer U14.11 (D3)
- net BUS6: now also U14.11 (D3); no longer U14.14 (D5)
- net Q0: now also U19.14 (I6); no longer U19.6 (I3)
- net Q1: now also U19.12 (I5); no longer U19.4 (I2)
- net Q2: now also U19.10 (I4); no longer U19.2 (I1)
- net Q3: now also U19.6 (I3); no longer U19.14 (I6)
- net Q4: now also U19.4 (I2); no longer U19.12 (I5)
- net Q5: now also U19.2 (I1); no longer U19.10 (I4)
Changed lines of the file:
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@@
   (junction (at 80.01 49.53) (diameter 0) (color 0 0 0 0)
   )
-  (wire (pts (xy 57.15 66.04) (xy 57.15 71.12))
-    (stroke (width 0) (type default))
-  )
-  (wire (pts (xy 49.53 62.23) (xy 49.53 66.04))
-    (stroke (width 0) (type default))
-  )
-  (wire (pts (xy 54.61 64.77) (xy 50.8 64.77))
-    (stroke (width 0) (type default))
-  )
-  (wire (pts (xy 62.23 62.23) (xy 62.23 66.04))
-    (stroke (width 0) (type default))
-  )
-  (wire (pts (xy 54.61 66.04) (xy 54.61 71.12))
-    (stroke (width 0) (type default))
-  )
   (wire (pts (xy 41.91 41.91) (xy 41.91 49.53))
-    (stroke (width 0) (type default))
-  )
-  (wire (pts (xy 50.8 71.12) (xy 49.53 71.12))
-    (stroke (width 0) (type default))
-  )
-  (wire (pts (xy 60.96 71.12) (xy 62.23 71.12))
-    (stroke (width 0) (type default))
-  )
-  (wire (pts (xy 49.53 66.04) (xy 54.61 66.04))
     (stroke (width 0) (type default))
   )
@@
     (stroke (width 0) (type default))
   )
-  (wire (pts (xy 52.07 71.12) (xy 52.07 62.23))
-    (stroke (width 0) (type default))
-  )
-  (wire (pts (xy 62.23 66.04) (xy 57.15 66.04))
-    (stroke (width 0) (type default))
-  )
   (wire (pts (xy 69.85 71.12) (xy 72.39 71.12))
-    (stroke (width 0) (type default))
-  )
-  (wire (pts (xy 54.61 62.23) (xy 54.61 64.77))
     (stroke (width 0) (type default))
   )
@@
     (stroke (width 0) (type default))
   )
-  (wire (pts (xy 57.15 62.23) (xy 57.15 64.77))
-    (stroke (width 0) (type default))
-  )
   (wire (pts (xy 80.01 41.91) (xy 80.01 49.53))
-    (stroke (width 0) (type default))
-  )
-  (wire (pts (xy 60.96 64.77) (xy 60.96 71.12))
-    (stroke (width 0) (type default))
-  )
-  (wire (pts (xy 59.69 71.12) (xy 59.69 62.23))
-    (stroke (width 0) (type default))
-  )
-  (wire (pts (xy 57.15 64.77) (xy 60.96 64.77))
     (stroke (width 0) (type default))
   )
@@
     (stroke (width 0) (type default))
   )
-  (wire (pts (xy 50.8 64.77) (xy 50.8 71.12))
-    (stroke (width 0) (type default))
-  )
-  (label "Q3" (at 57.15 63.5 90) (fields_autoplaced)
+  (label "Q3" (at 54.61 71.12 90) (fields_autoplaced)
     (effects (font (size 1.27 1.27)) (justify left bottom))
   )
-  (label "Q4" (at 59.69 63.5 90) (fields_autoplaced)
+  (label "Q0" (at 62.23 71.12 90) (fields_autoplaced)
     (effects (font (size 1.27 1.27)) (justify left bottom))
   )
-  (label "Q1" (at 52.07 63.5 90) (fields_autoplaced)
+  (label "Q5" (at 49.53 71.12 90) (fields_autoplaced)
     (effects (font (size 1.27 1.27)) (justify left bottom))
   )
-  (label "Q2" (at 54.61 63.5 90) (fields_autoplaced)
+  (label "Q2" (at 57.15 71.12 90) (fields_autoplaced)
     (effects (font (size 1.27 1.27)) (justify left bottom))
   )
-  (label "Q0" (at 49.53 63.5 90) (fields_autoplaced)
+  (label "Q3" (at 57.15 62.23 90) (fields_autoplaced)
     (effects (font (size 1.27 1.27)) (justify left bottom))
   )
-  (label "Q5" (at 62.23 63.5 90) (fields_autoplaced)
+  (label "Q4" (at 59.69 62.23 90) (fields_autoplaced)
+    (effects (font (size 1.27 1.27)) (justify left bottom))
+  )
+  (label "Q1" (at 52.07 62.23 90) (fields_autoplaced)
+    (effects (font (size 1.27 1.27)) (justify left bottom))
+  )
+  (label "Q2" (at 54.61 62.23 90) (fields_autoplaced)
+    (effects (font (size 1.27 1.27)) (justify left bottom))
+  )
+  (label "Q0" (at 49.53 62.23 90) (fields_autoplaced)
+    (effects (font (size 1.27 1.27)) (justify left bottom))
+  )
+  (label "Q5" (at 62.23 62.23 90) (fields_autoplaced)
+    (effects (font (size 1.27 1.27)) (justify left bottom))
+  )
+  (label "Q1" (at 59.69 71.12 90) (fields_autoplaced)
+    (effects (font (size 1.27 1.27)) (justify left bottom))
+  )
+  (label "Q4" (at 52.07 71.12 90) (fields_autoplaced)
     (effects (font (size 1.27 1.27)) (justify left bottom))
   )
@@
     (effects (font (size 1.27 1.27)) (justify right))
   )
-  (hierarchical_label "BUS4" (shape input) (at 57.15 36.83 90) (fields_autoplaced)
-    (effects (font (size 1.27 1.27)) (justify left))
-  )
   (hierarchical_label "BUS5" (shape input) (at 59.69 36.83 90) (fields_autoplaced)
     (effects (font (size 1.27 1.27)) (justify left))
@@
     (effects (font (size 1.27 1.27)) (justify right))
   )
+  (hierarchical_label "BUS1" (shape input) (at 54.61 36.83 90) (fields_autoplaced)
+    (effects (font (size 1.27 1.27)) (justify left))
+  )
+  (hierarchical_label "BUS6" (shape input) (at 57.15 36.83 90) (fields_autoplaced)
+    (effects (font (size 1.27 1.27)) (justify left))
+  )
   (hierarchical_label "L5" (shape input) (at 59.69 96.52 270) (fields_autoplaced)
     (effects (font (size 1.27 1.27)) (justify right))
-  )
-  (hierarchical_label "BUS6" (shape input) (at 62.23 36.83 90) (fields_autoplaced)
-    (effects (font (size 1.27 1.27)) (justify left))
   )
   (hierarchical_label "BUS2" (shape input) (at 52.07 36.83 90) (fields_autoplaced)
     (effects (font (size 1.27 1.27)) (justify left))
   )
-  (hierarchical_label "BUS1" (shape input) (at 49.53 36.83 90) (fields_autoplaced)
+  (hierarchical_label "R" (shape input) (at 72.39 36.83 90) (fields_autoplaced)
     (effects (font (size 1.27 1.27)) (justify left))
   )
-  (hierarchical_label "R" (shape input) (at 72.39 36.83 90) (fields_autoplaced)
+  (hierarchical_label "BUS4" (shape input) (at 62.23 36.83 90) (fields_autoplaced)
+    (effects (font (size 1.27 1.27)) (justify left))
+  )
+  (hierarchical_label "BUS3" (shape input) (at 49.53 36.83 90) (fields_autoplaced)
     (effects (font (size 1.27 1.27)) (justify left))
   )
@@
     (effects (font (size 1.27 1.27)) (justify left))
   )
-  (hierarchical_label "BUS3" (shape input) (at 54.61 36.83 90) (fields_autoplaced)
-    (effects (font (size 1.27 1.27)) (justify left))
-  )

Commit message: Finalize the board
Parts:
- U14, U19: footprint Package_SO:TSSOP-16_4.4x5mm_P0.65mm -> GKanwarLibrary:TSSOP-16_4.4x5mm_P0.65mm
Changed lines of the file:
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@@
       (effects (font (size 1.27 1.27)))
     )
-    (property "Footprint" "Package_SO:TSSOP-16_4.4x5mm_P0.65mm" (at 59.69 83.82 0)
+    (property "Footprint" "GKanwarLibrary:TSSOP-16_4.4x5mm_P0.65mm" (at 59.69 83.82 0)
       (effects (font (size 1.27 1.27)) hide)
     )
@@
       (effects (font (size 1.27 1.27)))
     )
-    (property "Footprint" "Package_SO:TSSOP-16_4.4x5mm_P0.65mm" (at 59.69 49.53 0)
+    (property "Footprint" "GKanwarLibrary:TSSOP-16_4.4x5mm_P0.65mm" (at 59.69 49.53 0)
       (effects (font (size 1.27 1.27)) hide)
     )

Commit message: readme: Added with many images and a snippet of the timelapse
Parts:
- renumbered U14 to U13
