File: unchat_keeb/right_switches.kicad_sch (KiCad schematic)
At the start: 54 parts

Commit message: Add extra columns, updating to 42-key design
Parts:
- added L10, L15, L5: LED, LED_SMD:LED_0603_1608Metric, symbol Device:LED_Small
- added R77, R82, R87: 100, Resistor_SMD:R_0805_2012Metric, symbol ScottoKeebs:Placeholder_Resistor
- added S? (x3): Keyswitch, GKanwarLibrary:Choc_V1_LED_1.00u, symbol ScottoKeebs:Placeholder_Keyswitch
Connections:
- net GND: now also R77.1, R82.1, R87.1
- net L1: now also L5.1 (K); no longer L5.1 (K)
- net L10: now also L8.1 (K); no longer L6.1 (K)
- net L11: now also L7.1 (K); no longer L15.1 (K)
- net L12: now also L6.1 (K); no longer L14.1 (K)
- net L13: now also L15.1 (K); no longer L13.1 (K)
- net L14: now also L15.1 (K); no longer L12.1 (K)
- net L15: now also L14.1 (K); no longer L11.1 (K)
- net L16: now also L13.1 (K); no longer L18.1 (K)
- net L17: now also L12.1 (K); no longer L17.1 (K)
- net L18: now also L11.1 (K); no longer L16.1 (K)
- net L2: now also L5.1 (K); no longer L4.1 (K)
- net L3: now also L4.1 (K); no longer L3.1 (K)
- net L4: now also L3.1 (K); no longer L2.1 (K)
- net L5: now also L2.1 (K); no longer L1.1 (K)
- net L6: now also L1.1 (K); no longer L10.1 (K)
- net L7: now also L10.1 (K); no longer L9.1 (K)
- net L8: now also L10.1 (K); no longer L8.1 (K)
- net L9: now also L9.1 (K); no longer L7.1 (K)
- net S10a: now also S?.1; no longer S?.1
- net S10b: now also S?.2; no longer S?.2
- net S11a: now also S?.1; no longer S?.1
- net S11b: now also S?.2; no longer S?.2
- net S12a: now also S?.1; no longer S?.1
- net S12b: now also S?.2; no longer S?.2
- net S13a: now also S?.1; no longer S?.1
- net S13b: now also S?.2; no longer S?.2
- net S14a: now also S?.1; no longer S?.1
- net S14b: now also S?.2; no longer S?.2
- net S15a: now also S?.1; no longer S?.1
- net S15b: now also S?.2; no longer S?.2
- net S16a: now also S?.1; no longer S?.1
- net S16b: now also S?.2; no longer S?.2
- net S17a: now also S?.1; no longer S?.1
- net S17b: now also S?.2; no longer S?.2
- net S18a: now also S?.1; no longer S?.1
- net S18b: now also S?.2; no longer S?.2
- net S1a: now also S?.1; no longer S?.1
- net S1b: now also S?.2; no longer S?.2
- net S2a: now also S?.1; no longer S?.1
- net S2b: now also S?.2; no longer S?.2
- net S3a: now also S?.1; no longer S?.1
- net S3b: now also S?.2; no longer S?.2
- net S4a: now also S?.1; no longer S?.1
- net S4b: now also S?.2; no longer S?.2
- net S5a: now also S?.1; no longer S?.1
- net S5b: now also S?.2; no longer S?.2
- net S6a: now also S?.1; no longer S?.1
- net S6b: now also S?.2; no longer S?.2
- net S7a: now also S?.1; no longer S?.1
- net S7b: now also S?.2; no longer S?.2
- net S8a: now also S?.1; no longer S?.1
- net S8b: now also S?.2; no longer S?.2
- net S9a: now also S?.1; no longer S?.1
- net S9b: now also S?.2; no longer S?.2
- new net: L15.2 (A), R87.2
- new net: L10.2 (A), R82.2
- new net: L5.2 (A), R77.2
- new net L19: L18.1 (K)
- new net L20: L17.1 (K)
- new net L21: L16.1 (K)
- new net S19a: S?.1
- new net S19b: S?.2
- new net S20a: S?.1
- new net S20b: S?.2
- new net S21a: S?.1
- new net S21b: S?.2
Other:
- moved on the sheet: S?

Commit message: readme: Added with many images and a snippet of the timelapse
Parts:
- gave numbers to parts that had none: 21
- renumbered L5 to L22, L5 to L23, L4 to L24, L3 to L25, L2 to L26, L1 to L27, L10 to L28, L10 to L29, L9 to L30, L8 to L31, L7 to L32, L6 to L33, L15 to L34, L15 to L35, L14 to L36, L13 to L39, L12 to L40, L11 to L41, L18 to L42, L17 to L43, L16 to L44, R80 to R100, R79 to R101, R78 to R102, R87 to R103, R87 to R104, R86 to R105, R85 to R106, R84 to R107, R83 to R108, R90 to R114, R89 to R115, R88 to R116, R77 to R91, R77 to R92, R76 to R93, R75 to R94, R74 to R95, R73 to R96, R82 to R97, R82 to R98, R81 to R99
