File: unchat_keeb_v2/unchat_keeb_v2.kicad_pcb (KiCad board)
At the start: 2 copper layers, 141.8 x 86.9 mm, 89 parts, among them J1 RJ45, J51 RJ45, U1 DRV5055, U10 DRV5055, U11 DRV5055, U12 DRV5055, U13 DRV5055, U14 DRV5055, U15 DRV5055, U16 DRV5055, U17 DRV5055, U18 DRV5055, U19 DRV5055, U2 DRV5055, U20 DRV5055, U22 CD74HC4067SM, U23 CD74HC4067SM, U3 DRV5055, U4 DRV5055, U5 DRV5055, U51 DRV5055, U52 DRV5055, U53 DRV5055, U54 DRV5055, U55 DRV5055, U56 DRV5055, U57 DRV5055, U58 DRV5055, U59 DRV5055, U6 DRV5055, U60 DRV5055, U61 DRV5055, U62 DRV5055, U63 DRV5055, U64 DRV5055, U65 DRV5055, U66 DRV5055, U67 DRV5055, U68 DRV5055, U69 DRV5055, U7 DRV5055, U70 DRV5055, U72 CD74HC4067SM, U73 CD74HC4067SM, U8 DRV5055, U9 DRV5055

Commit message: readme: Added with many images and a snippet of the timelapse
Changed lines of the file:
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@@
 		(polygon
 			(pts
-				(xy 72.5 47.5) (xy 72.5 115) (xy 122.5 115) (xy 140 135) (xy 185 140) (xy 217.5 112.5) (xy 217.5 47.5)
+				(xy 69.8 45.2) (xy 69 145.1) (xy 225.9 145.5) (xy 226.1 45.4)
 			)
 		)
